Commit message: urdf mass updates

File: alexander-models/alexander_V1_description/urdf/alexander_v1.lowerBody.urdf (robot description, URDF)
Before this commit: robot Alexander, 24 links, 23 joints
Links:
- link LEFT_FOOT: mass 1.28288609 -> 1.314
- link LEFT_HIP_X_LINK: mass 2.32977961 -> 1.933
- link LEFT_HIP_Z_LINK: mass 0.77281362 -> 0.777
- link LEFT_SHIN: mass 5.5 -> 7.400
- link LEFT_THIGH: mass 7.75 -> 8.200
- link PELVIS_LINK: mass 9.50083635 -> 7.700
- link RIGHT_FOOT: mass 1.28288609 -> 1.314
- link RIGHT_HIP_X_LINK: mass 2.32977248 -> 1.933
- link RIGHT_HIP_Z_LINK: mass 0.77281055 -> 0.777
- link RIGHT_SHIN: mass 5.5 -> 7.400
- link RIGHT_THIGH: mass 7.75 -> 8.200

Commit message: Mass and Inertias are updated from measured mass

File: alexander-models/alexander_V1_description/urdf/alexander_v1.lowerBody.urdf (robot description, URDF)
Before this commit: robot Alexander, 24 links, 23 joints
Links:
- link LEFT_ANKLE_Y_LINK: mass 0.05045632 -> 0.04972436486
- link LEFT_FOOT: mass 1.314 -> 1.264275635
- link RIGHT_ANKLE_Y_LINK: mass 0.05045632 -> 0.04972436486
- link RIGHT_FOOT: mass 1.314 -> 1.264275635
- link TORSO_LINK: mass 4.208 -> 2.13269743

File: alexander-models/alexander_V1_description/urdf/alexander_v1.lowerBodyOnly.urdf (robot description, URDF)
Before this commit: robot Alexander, 23 links, 22 joints
Links:
- link LEFT_ANKLE_Y_LINK: mass 0.05045632 -> 0.04972436486
- link LEFT_FOOT: mass 1.28288609 -> 1.264275635
- link LEFT_HIP_X_LINK: mass 2.32977961 -> 1.933
- link LEFT_HIP_Z_LINK: mass 0.77281362 -> 0.777
- link LEFT_SHIN: mass 5.5 -> 7.400
- link LEFT_THIGH: mass 7.75 -> 8.200
- link PELVIS_LINK: mass 9.50083635 -> 7.700
- link RIGHT_ANKLE_Y_LINK: mass 0.05045632 -> 0.04972436486
- link RIGHT_FOOT: mass 1.28288609 -> 1.264275635
- link RIGHT_HIP_X_LINK: mass 2.32977248 -> 1.933
- link RIGHT_HIP_Z_LINK: mass 0.77281055 -> 0.777
- link RIGHT_SHIN: mass 5.5 -> 7.400
- link RIGHT_THIGH: mass 7.75 -> 8.200
- link TORSO_LINK: mass 4.208 -> 2.13269743
