Commit message: Remove trailing whitespace in some URDF entries

File: alexander-models/alexander_V1_description/urdf/alexander_v1.fullBody.urdf (robot description, URDF)
Before this commit: robot Alexander, 41 links, 40 joints
Joints:
- joint LEFT_HIP_X: limit lower=-0.3490658504  upper=0.872664626 effort=150 velocity=9 -> lower=-0.3490658504 upper=0.872664626 effort=150 velocity=9

File: alexander-models/alexander_V1_description/urdf/alexander_v1.lowerBody.urdf (robot description, URDF)
Before this commit: robot Alexander, 24 links, 23 joints
Joints:
- joint LEFT_HIP_X: limit lower=-0.3490658504  upper=0.872664626 effort=150 velocity=9 -> lower=-0.3490658504 upper=0.872664626 effort=150 velocity=9

File: alexander-models/alexander_V1_description/urdf/alexander_v1.lowerBodyOnly.urdf (robot description, URDF)
Before this commit: robot Alexander, 23 links, 22 joints
Joints:
- joint LEFT_HIP_X: limit lower=-0.3490658504  upper=0.872664626 effort=150 velocity=9 -> lower=-0.3490658504 upper=0.872664626 effort=150 velocity=9

Commit message: Refactor URDFs, include new GLBs, remove .g3djs.

File: alexander-models/alexander_V1_description/urdf/alexander_v1.fullBody.urdf (robot description, URDF)
Before this commit: robot Alexander, 41 links, 40 joints
Links:
- link LEFT_ANKLE_Y_LINK: geometry visual mesh filename=package://alexander_V1_description/meshes/legs/AnklePitchLi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
- link LEFT_FOOT: geometry visual mesh filename=package://alexander_V1_description/meshes/legs/Foot.obj
- link LEFT_THIGH: geometry visual mesh filename=package://alexander_V1_description/meshes/legs/LeftThigh.obj
- link RIGHT_ANKLE_Y_LINK: geometry visual mesh filename=package://alexander_V1_description/meshes/legs/AnklePitchLi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
- link RIGHT_FOOT: geometry visual mesh filename=package://alexander_V1_description/meshes/legs/Foot.obj
- link RIGHT_THIGH: geometry visual mesh filename=package://alexander_V1_description/meshes/legs/RightThigh.o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

File: alexander-models/alexander_V1_description/urdf/alexander_v1.lowerBody.urdf (robot description, URDF)
Before this commit: robot Alexander, 24 links, 23 joints
Links:
- link LEFT_ANKLE_Y_LINK: geometry visual mesh filename=package://alexander_V1_description/meshes/legs/AnklePitchLi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
- link LEFT_FOOT: geometry visual mesh filename=package://alexander_V1_description/meshes/legs/Foot.obj
- link LEFT_THIGH: geometry visual mesh filename=package://alexander_V1_description/meshes/legs/LeftThigh.obj
- link RIGHT_ANKLE_Y_LINK: geometry visual mesh filename=package://alexander_V1_description/meshes/legs/AnklePitchLi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
- link RIGHT_FOOT: geometry visual mesh filename=package://alexander_V1_description/meshes/legs/Foot.obj
- link RIGHT_THIGH: geometry visual mesh filename=package://alexander_V1_description/meshes/legs/RightThigh.o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

File: alexander-models/alexander_V1_description/urdf/alexander_v1.lowerBodyOnly.urdf (robot description, URDF)
Before this commit: robot Alexander, 23 links, 22 joints
Links:
- link LEFT_ANKLE_Y_LINK: geometry visual mesh filename=package://alexander_V1_description/meshes/legs/AnklePitchLi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
- link LEFT_FOOT: geometry visual mesh filename=package://alexander_V1_description/meshes/legs/Foot.obj
- link LEFT_THIGH: geometry visual mesh filename=package://alexander_V1_description/meshes/legs/LeftThigh.obj
- link RIGHT_ANKLE_Y_LINK: geometry visual mesh filename=package://alexander_V1_description/meshes/legs/AnklePitchLi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
- link RIGHT_FOOT: geometry visual mesh filename=package://alexander_V1_description/meshes/legs/Foot.obj
- link RIGHT_THIGH: geometry visual mesh filename=package://alexander_V1_description/meshes/legs/RightThigh.o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

Commit message: Adding reduced poly meshes

File: alexander-models/alexander_V1_description/urdf/alexander_v1.fullBody.urdf (robot description, URDF)
Before this commit: robot Alexander, 41 links, 40 joints
Links:
- link LEFT_ANKLE_Y_LINK: geometry visual mesh filename=package://alexander_V1_description/meshes/legs/AnklePitchLi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
- link LEFT_FOOT: geometry visual mesh filename=package://alexander_V1_description/meshes/legs/Foot.obj
- link LEFT_SHIN: geometry visual mesh filename=package://alexander_V1_description/meshes/legs/LeftShin.obj
- link LEFT_THIGH: geometry visual mesh filename=package://alexander_V1_description/meshes/legs/LeftThigh.obj
- link RIGHT_ANKLE_Y_LINK: geometry visual mesh filename=package://alexander_V1_description/meshes/legs/AnklePitchLi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
- link RIGHT_FOOT: geometry visual mesh filename=package://alexander_V1_description/meshes/legs/Foot.obj
- link RIGHT_SHIN: geometry visual mesh filename=package://alexander_V1_description/meshes/legs/RightShin.obj
- link RIGHT_THIGH: geometry visual mesh filename=package://alexander_V1_description/meshes/legs/RightThigh.o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

File: alexander-models/alexander_V1_description/urdf/alexander_v1.lowerBodyOnly.urdf (robot description, URDF)
Before this commit: robot Alexander, 23 links, 22 joints
Links:
- link LEFT_ANKLE_Y_LINK: geometry visual mesh filename=package://alexander_V1_description/meshes/legs/AnklePitchLi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
- link LEFT_FOOT: geometry visual mesh filename=package://alexander_V1_description/meshes/legs/Foot.obj
- link LEFT_SHIN: geometry visual mesh filename=package://alexander_V1_description/meshes/legs/LeftShin.obj
- link LEFT_THIGH: geometry visual mesh filename=package://alexander_V1_description/meshes/legs/LeftThigh.obj
- link RIGHT_ANKLE_Y_LINK: geometry visual mesh filename=package://alexander_V1_description/meshes/legs/AnklePitchLi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
- link RIGHT_FOOT: geometry visual mesh filename=package://alexander_V1_description/meshes/legs/Foot.obj
- link RIGHT_SHIN: geometry visual mesh filename=package://alexander_V1_description/meshes/legs/RightShin.obj
- link RIGHT_THIGH: geometry visual mesh filename=package://alexander_V1_description/meshes/legs/RightThigh.o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
